Commit message: camera viwer and replay

File: simulation/infobot_agent/urdf/properties.xacro (robot description, xacro)
@@ -2,5 +2,5 @@
 <robot xmlns:xacro="http://ros.org/wiki/xacro">
 <!-- GOPAL400 and FORKLIFT -->
-<xacro:property name="robot_type" value="FORKLIFT"/>
+<xacro:property name="robot_type" value="GOPAL400"/>
     <xacro:property name="base_length" value="1.4"/>
     <xacro:property name="base_width" value="0.86"/> <!-- wheel_separation -->
@@ -21,6 +21,6 @@
     <xacro:property name="infobot_damping" value="0.7"/>
     <xacro:property name="infobot_slide_range" value="2"/>
+<!--GOPAL 400 :  https://www.mobile-robots.de/files/554/factsheet-mr-robotize-gopal-400-e24-09-22-en-min.pdf -->
 <xacro:if value="${robot_type == 'GOPAL400'}">
-    <!--GOPAL 400 :  https://www.mobile-robots.de/files/554/factsheet-mr-robotize-gopal-400-e24-09-22-en-min.pdf -->
     <xacro:property name="fork_size_x" value="1.2"/>
     <xacro:property name="fork_size_y" value="0.1"/>
@@ -30,6 +30,6 @@
     <xacro:property name="fork_pos_z" value="0.0"/>
 </xacro:if>
+<!-- FORKLIFT -->
 <xacro:if value="${robot_type == 'FORKLIFT'}">
-    <!-- FORKLIFT -->
     <xacro:property name="fork_size_x" value="1.2"/>
     <xacro:property name="fork_size_y" value="0.1"/>

File: simulation/static_agent_launcher/description/camera_config.xacro (robot description, xacro)
@@ -2,15 +2,15 @@
 <!-- =================================== -->
 <robot xmlns:xacro="http://www.ros.org/wiki/xacro">
-<xacro:camera number="160" x="-23.768993347281643" y="1.095911585638125" z="7.792710237230575" r="-3.072200475262292" p="2.0401256682927498" w="3.1384164986805017" width="216" height="384" k1="0" k2="0" k3="0" p1="0" p2="0" horizental_fov="1"  />
-<xacro:camera number="161" x="-15.548574448619283" y="1.1875803973838794" z="8.430721825553768" r="3.1401165362282915" p="1.8467776536834755" w="-3.075174579490206" width="216" height="384" k1="0" k2="0" k3="0" p1="0" p2="0" horizental_fov="1"  />
-<xacro:camera number="162" x="-5.583158189893617" y="1.1215696998181661" z="7.334558192411435" r="-3.121470473216963" p="1.882414969291388" w="3.1315374728737932" width="216" height="384" k1="0" k2="0" k3="0" p1="0" p2="0" horizental_fov="1"  />
-<xacro:camera number="163" x="6.408863223463873" y="1.0584660310604614" z="7.292500745934432" r="-3.1247537437337134" p="1.6132230097420674" w="3.072926607602098" width="216" height="384" k1="0" k2="0" k3="0" p1="0" p2="0" horizental_fov="1"  />
-<xacro:camera number="164" x="19.018611699231805" y="0.5996158690202327" z="7.312413251033552" r="3.0865049949744816" p="1.2064798251635096" w="-0.10259603486110593" width="216" height="384" k1="0" k2="0" k3="0" p1="0" p2="0" horizental_fov="1"  />
-<xacro:camera number="165" x="19.780977546074062" y="-3.5988921587419385" z="7.320450325717854" r="3.092351302733551" p="1.9069402784416059" w="-1.63895299731986" width="216" height="384" k1="0" k2="0" k3="0" p1="0" p2="0" horizental_fov="1"  />
-<xacro:camera number="166" x="22.963270174027638" y="4.027979359238905" z="7.419277685692496" r="-2.9569181358814967" p="1.5216930354201401" w="-2.3427224426882813" width="216" height="384" k1="0" k2="0" k3="0" p1="0" p2="0" horizental_fov="1"  />
-<xacro:camera number="167" x="20.320795688398483" y="8.551222492793519" z="7.698006516690173" r="-2.864067809004126" p="1.6165247062294361" w="3.049326481704911" width="216" height="384" k1="0" k2="0" k3="0" p1="0" p2="0" horizental_fov="1"  />
-<xacro:camera number="168" x="26.791802520963806" y="5.716299217374743" z="3.8958341874803013" r="2.0879686599511014" p="1.5484721682976101" w="0.02430880840685812" width="216" height="384" k1="0" k2="0" k3="0" p1="0" p2="0" horizental_fov="1"  />
-<xacro:camera number="169" x="30.084965589192375" y="9.359551955197704" z="5.179745027009818" r="-2.6817009758316908" p="1.442123361726637" w="-3.087108573615953" width="216" height="384" k1="0" k2="0" k3="0"  p1="0" p2="0"  horizental_fov="1"  />
-<xacro:camera number="170" x="36.82995339051741" y="9.404901482485903" z="5.154350415603337" r="-2.66777470309351" p="1.5376363780888378" w="-3.089363397883026" width="216" height="384" k1="0" k2="0" k3="0" p1="0" p2="0"  horizental_fov="1"  />
-<xacro:camera number="171" x="42.44269046560321" y="9.38157274756824" z="5.146596979178394" r="-2.7448623326295176" p="1.5704089535445784" w="-3.132973283776775" width="216" height="384" k1="0" k2="0" k3="0" p1="0" p2="0" horizental_fov="1"  />
+<xacro:camera number="160" x="-23.768993347281643" y="1.0959115856381252" z="7.792710237230576" r="-3.072200475262292" p="2.0401256682927498" w="3.1384164986805017" width="2160" height="3840" k1="-0.3990864717265948" k2="0.2016451846353012" k3="-0.053753317426588856" p1="-0.00013457492654973615" p2="0.0003788431220127677" horizental_fov="0.9062245961423843" aspect_ratio="0.6346135746416991"  />
+<xacro:camera number="161" x="-15.54857444861928" y="1.1875803973838794" z="8.430721825553768" r="3.1401165362282915" p="1.8467776536834755" w="-3.075174579490206" width="2160" height="3840" k1="-0.5337684959685228" k2="0.34369206124627594" k3="-0.11312322233867529" p1="-0.001568761626559521" p2="0.0012933658245218613" horizental_fov="0.7979068207653639" aspect_ratio="0.6219373044342069"  />
+<xacro:camera number="162" x="-5.583158189893618" y="1.1215696998181661" z="7.334558192411434" r="-3.121470473216963" p="1.882414969291388" w="3.1315374728737932" width="2160" height="3840" k1="-0.3881529379410545" k2="0.21282043348416652" k3="-0.07191487688493671" p1="7.348232914337802e-05" p2="-0.0003723515252576787" horizental_fov="0.934637563021535" aspect_ratio="0.6380980311690627"  />
+<xacro:camera number="163" x="6.408863223463874" y="1.0584660310604614" z="7.292500745934433" r="-3.1247537437337134" p="1.6132230097420674" w="3.072926607602098" width="2160" height="3840" k1="-0.38583566587127305" k2="0.2099961443873393" k3="-0.07094931776988343" p1="0.00014849011979552266" p2="9.279371221442497e-05" horizental_fov="0.9312481766450852" aspect_ratio="0.6378137006195269"  />
+<xacro:camera number="164" x="19.018611699231805" y="0.5996158690202326" z="7.312413251033551" r="3.0865049949744816" p="1.2064798251635096" w="-0.10259603486110593" width="2160" height="3840" k1="-0.3851544658419547" k2="0.2065606446662026" k3="-0.06703301309031716" p1="-0.0002282099854856601" p2="-8.882469357164693e-05" horizental_fov="0.9343447506168914" aspect_ratio="0.6383050770452745"  />
+<xacro:camera number="165" x="19.780977546074062" y="-3.598892158741938" z="7.320450325717852" r="3.092351302733551" p="1.9069402784416059" w="-1.63895299731986" width="2160" height="3840" k1="-0.3856199901471728" k2="0.20812766168662827" k3="-0.0686518264523881" p1="-8.229104930400743e-05" p2="-0.00023961544692403472" horizental_fov="0.9339854982138229" aspect_ratio="0.6382418389072573"  />
+<xacro:camera number="166" x="22.963270174027635" y="4.027979359238904" z="7.419277685692497" r="-2.9569181358814967" p="1.5216930354201401" w="-2.3427224426882813" width="2160" height="3840" k1="-0.38144336503488374" k2="0.19579882600150705" k3="-0.0586530291683016" p1="-2.68226954291596e-05" p2="-0.0002683294214338217" horizental_fov="0.9341965766788635" aspect_ratio="0.6380356409363908"  />
+<xacro:camera number="167" x="20.320795688398483" y="8.551222492793519" z="7.698006516690173" r="-2.864067809004126" p="1.6165247062294361" w="3.049326481704911" width="2160" height="3840" k1="-0.3838819131967851" k2="0.2010505063378464" k3="-0.062406328638322184" p1="-0.0001711681317662323" p2="-0.0001384477473404489" horizental_fov="0.9326674829664602" aspect_ratio="0.6380360618380091"  />
+<xacro:camera number="168" x="26.79180252096381" y="5.716299217374743" z="3.8958341874803013" r="2.0879686599511014" p="1.5484721682976101" w="0.02430880840685812" width="2160" height="3840" k1="-0.38226542199738556" k2="0.19688945293158802" k3="-0.05884113267485558" p1="-0.00019454336997989425" p2="0.00010222372875181348" horizental_fov="0.930340781288024" aspect_ratio="0.6377205101360616"  />
+<xacro:camera number="169" x="30.084965589192375" y="9.359551955197704" z="5.17974502700982" r="-2.6817009758316908" p="1.442123361726637" w="-3.087108573615953" width="2160" height="3840" k1="-0.376908078697939" k2="0.1841695668036844" k3="-0.05236396951447785" p1="-0.0006789329541068425" p2="-0.0003816943552840085" horizental_fov="0.9306534293111707" aspect_ratio="0.6373718963712801"  />
+<xacro:camera number="170" x="36.82995339051741" y="9.404901482485904" z="5.154350415603337" r="-2.66777470309351" p="1.5376363780888378" w="-3.089363397883026" width="2160" height="3840" k1="-0.3840696848810335" k2="0.20309686574554098" k3="-0.06443293775304995" p1="-0.0002648898125099341" p2="0.00011495455326132926" horizental_fov="0.9336309514986754" aspect_ratio="0.6382016868830621"  />
+<xacro:camera number="171" x="42.4426904656032" y="9.38157274756824" z="5.146596979178394" r="-2.7448623326295176" p="1.5704089535445784" w="-3.132973283776775" width="2160" height="3840" k1="-0.3840696848810335" k2="0.20309686574554098" k3="-0.06443293775304995" p1="-0.0002648898125099341" p2="0.00011495455326132926" horizental_fov="0.9336309514986754" aspect_ratio="0.6382016868830621"  />
 </robot>

File: simulation/static_agent_launcher/description/camera_macros.xacro (robot description, xacro)
@@ -24,12 +24,13 @@
         </joint>
     </xacro:macro>
-    <xacro:macro name="camera_gazebo" params="number width height k1 k2 k3 p1 p2 horizental_fov">
+    <xacro:macro name="camera_gazebo" params="number width height k1 k2 k3 p1 p2 horizental_fov aspect_ratio">
         <gazebo reference="camera_${number}_link">
             <sensor name="camera_${number}" type="camera">
                 <always_on>true</always_on>
                 <visualize>true</visualize>
-                <update_rate>1</update_rate>
+                <update_rate>0</update_rate>
                 <camera name="intel_realsense_r200">
                   <horizontal_fov>${horizental_fov}</horizontal_fov>
+                  <aspect_ratio>${aspect_ratio}</aspect_ratio>
                   <image>
                     <width>${width}</width>
@@ -37,4 +38,5 @@
                     <format>R8G8B8</format>
                   </image>
+<!--
                   <clip>
                     <near>0.02</near>
@@ -46,4 +48,5 @@
                     <stddev>0.007</stddev>
                   </noise>
+-->
                     <distortion>
                         <k1>${k1}</k1>
@@ -59,8 +62,8 @@
         </gazebo>
     </xacro:macro>
-    <xacro:macro name="camera" params="number x y z r p w width height k1 k2 k3 p1 p2 horizental_fov">
+    <xacro:macro name="camera" params="number x y z r p w width height k1 k2 k3 p1 p2 horizental_fov aspect_ratio">
         <xacro:camera_link number="${number}"/>
         <xacro:camera_joint number="${number}" x="${x}" y="${y}" z="${z}" r="${r}" p="${p}" w="${w}"/>
-        <xacro:camera_gazebo number="${number}" width="${width}" height="${height}"    k1="${k1}" k2="${k2}" k3="${k3}" p1="${p1}" p2="${p2}" horizental_fov="${horizental_fov}"  />
+        <xacro:camera_gazebo number="${number}" width="${width}" height="${height}"    k1="${k1}" k2="${k2}" k3="${k3}" p1="${p1}" p2="${p2}" horizental_fov="${horizental_fov}" aspect_ratio="${aspect_ratio}"  />
     </xacro:macro>
 </robot>
