Commit message: new layout, ceiling cameras, GOPAL and forklift teleop and nav2

File: simulation/infobot_agent/urdf/infobot.gazebo.xacro (robot description, xacro)
@@ -8,5 +8,5 @@
     <xacro:macro name="gazebo_frictionless" params="ref">
         <gazebo reference="${ref}">
-            <material>Gazebo/Blue</material>
+            <material>Gazebo/Grey</material>
             <mu>0.0</mu>
             <mu2>0.0</mu2>
@@ -29,5 +29,5 @@
     <xacro:gazebo_withfriction ref="wheel_right_link" />
     <gazebo reference="base_link">
-        <material>Gazebo/Blue</material>
+        <material>Gazebo/Orange</material>
     </gazebo>
     <gazebo reference="imu_link">
@@ -191,8 +191,4 @@
       <joint_name>wheel_right_joint</joint_name>
     </plugin>
-    <!--
-    <xacro:include filename="/home/research/repositories/SMILEIV/simulation/install/static_agent_launcher/share/static_agent_launcher/description/aruco_macros.xacro" />
-    <xacro:attach_aruco attach_to="wheel_left_link" number="99" x="0" y="0" z="0.3" r="0" p="0" yw="0"/>
-    This doesn't work because aruco_macros.xacro is not present        -->
     </gazebo>
 </robot>

File: simulation/infobot_agent/urdf/joints.xacro (robot description, xacro)
@@ -6,5 +6,5 @@
             <child link="wheel_${prefix}_link" />
             <axis xyz="0 0 1" />
-            <origin xyz="${x} ${y} -${z}" rpy="0 ${pi/2} ${pi/2}" />
+            <origin xyz="${x} ${y} ${z}" rpy="0 ${pi/2} ${pi/2}" />
             <dynamics friction="0.0"/>
         </joint>
@@ -15,5 +15,5 @@
             <child link="wheel_${prefix}_link" />
             <axis xyz="0 0 1" />
-            <origin xyz="${x} ${y} -${z}" rpy="0 ${pi/2} ${pi/2}" />
+            <origin xyz="${x} ${y} ${z}" rpy="0 ${pi/2} ${pi/2}" />
             <dynamics friction="${infobot_friction}" damping="${infobot_damping}"/>
         </joint>
@@ -31,3 +31,125 @@
     <xacro:frictionless_wheel_joint_macro prefix="frictionless_front_left"  x="${(base_length/2 - wheel_radius) * -1}" y="${(base_width/2 - wheel_width) * 1}"   z="0" />
     <xacro:frictionless_wheel_joint_macro prefix="frictionless_front_right" x="${(base_length/2 - wheel_radius) * -1}" y="${(base_width/2 - wheel_width) * -1}"  z="0" />
+<!--
+ros2 topic pub /effort_controller/commands std_msgs/msg/Float64MultiArray "data:
+- -100"
+-->
+  <link name="slidebar">
+    <inertial>
+      <mass value="100"/>
+      <inertia ixx="1.0" ixy="0.0" ixz="0.0" iyy="1.0" iyz="0.0" izz="1.0"/>
+    </inertial>
+  </link>
+  <joint name="slidebar_to_base" type="fixed">
+    <origin rpy="0 0 0" xyz="0 0 1.28"/> <!-- IMPORTANT THIS HAS TO BE IN 0,0 TO KEEP THE ROBOT BALANCED-->
+    <parent link="base_link"/>
+    <child link="slidebar"/>
+  </joint>
+  <link name="cart">
+<xacro:if value="${robot_type == 'GOPAL400'}">
+    <visual>
+      <geometry>
+        <box size="${base_length} ${base_width} 0.03"/>
+      </geometry>
+      <origin xyz="0 0 0"/>
+    </visual>
+    <collision>
+      <geometry>
+        <box size="${base_length} ${base_width} 0.03"/>
+      </geometry>
+    </collision>
+</xacro:if>
+<xacro:if value="${robot_type == 'FORKLIFT'}">
+</xacro:if>
+    <inertial>
+      <mass value="1"/>
+      <inertia ixx="1.0" ixy="0.0" ixz="0.0" iyy="1.0" iyz="0.0" izz="1.0"/>
+    </inertial>
+  </link>
+  <joint name="slider_to_cart" type="prismatic">
+    <axis xyz=" 0 0 1"/>
+    <origin xyz="0.0 0.0 0.0"/>   <!-- position of the cart-->
+    <parent link="slidebar"/>
+    <child link="cart"/>
+    <limit effort="1000.0" lower="${infobot_slide_range / -2 }" upper="${infobot_slide_range /2 }" velocity="30"/>
+    <dynamics damping="0.0" friction="0.0"/>
+  </joint>
+  <gazebo reference="cart">
+    <material>Gazebo/Grey</material>
+  </gazebo>
+  <gazebo reference="fork1">
+    <material>Gazebo/DarkGrey</material>
+  </gazebo>
+  <gazebo reference="fork2">
+    <material>Gazebo/DarkGrey</material>
+  </gazebo>
+  <link name="fork1">
+    <visual>
+      <geometry>
+        <box size="${fork_size_x} ${fork_size_y} ${fork_size_z}"/>
+      </geometry>
+      <origin xyz="${fork_pos_x} ${fork_separation} ${fork_pos_z}"/>
+    </visual>
+    <collision>
+      <geometry>
+        <box size="${fork_size_x} ${fork_size_y} ${fork_size_z}"/>
+      </geometry>
+      <origin xyz="${fork_pos_x} ${fork_separation} ${fork_pos_z}"/>
+    </collision>
+    <inertial>
+      <mass value="0.01"/>
+      <inertia ixx="1.0" ixy="0.0" ixz="0.0" iyy="1.0" iyz="0.0" izz="1.0"/>
+    </inertial>
+  </link>
+  <joint name="fork1_to_cart" type="fixed">
+    <axis xyz=" 0 0 1"/>
+    <origin xyz="0 0 0"/>
+    <parent link="cart"/>
+    <child link="fork1"/>
+  </joint>
+  <link name="fork2">
+    <visual>
+      <geometry>
+        <box size="${fork_size_x} ${fork_size_y} ${fork_size_z}"/>
+      </geometry>
+      <origin xyz="${fork_pos_x} ${-1 * fork_separation} ${fork_pos_z}"/>
+    </visual>
+    <collision>
+      <geometry>
+        <box size="${fork_size_x} ${fork_size_y} ${fork_size_z}"/>
+      </geometry>
+      <origin xyz="${fork_pos_x} ${-1 * fork_separation} ${fork_pos_z}"/>
+    </collision>
+    <inertial>
+      <mass value="0.01"/>
+      <inertia ixx="1.0" ixy="0.0" ixz="0.0" iyy="1.0" iyz="0.0" izz="1.0"/>
+    </inertial>
+  </link>
+  <joint name="fork2_to_cart" type="fixed">
+    <axis xyz=" 0 0 1"/>
+    <origin xyz="0 0 0"/>
+    <parent link="cart"/>
+    <child link="fork2"/>
+  </joint>
+  <ros2_control name="GazeboSystem" type="system">
+    <hardware>
+      <plugin>gazebo_ros2_control/GazeboSystem</plugin>
+    </hardware>
+    <joint name="slider_to_cart">
+      <command_interface name="effort">
+        <param name="min">-1000</param>
+        <param name="max">1000</param>
+      </command_interface>
+      <state_interface name="position">
+        <param name="initial_value">0</param>
+      </state_interface>
+      <state_interface name="velocity"/>
+      <state_interface name="effort"/>
+    </joint>
+  </ros2_control>
+  <gazebo>
+    <plugin filename="libgazebo_ros2_control.so" name="gazebo_ros2_control">
+      <parameters>$(find infobot_agent)/config/controller_effort.yaml</parameters>
+    </plugin>
+  </gazebo>
 </robot>

File: simulation/infobot_agent/urdf/links.xacro (robot description, xacro)
@@ -4,4 +4,5 @@
     <link name="base_link">
         <visual>
+<xacro:if value="${robot_type == 'GOPAL400'}">
             <origin xyz="0 0 0" rpy="0 0 0" />
             <geometry>
@@ -9,11 +10,25 @@
                 <!-- <box size="${base_length} ${base_width} ${base_height}" /> -->
             </geometry>
-            <material name="blue"/>
+</xacro:if>
+<xacro:if value="${robot_type == 'FORKLIFT'}">
+            <origin xyz="-1.5 -0.5 0" rpy="0 0 0" />
+            <geometry>
+                <mesh filename="package://forklift_robot/forklift_robot_description/meshes/base_link.dae"/>
+            </geometry>
+</xacro:if>
         </visual>
         <collision>
+<xacro:if value="${robot_type == 'GOPAL400'}">
             <geometry>
                 <mesh filename="file://infobot_agent/models/infobot_common/meshes/AMR_GP400.dae" scale="1 1 1"/>
                 <!-- <box size="${base_length} ${base_width} ${base_height}" />  -->
             </geometry>
+</xacro:if>
+<xacro:if value="${robot_type == 'FORKLIFT'}">
+            <origin xyz="-1.5 -0.5 0" rpy="0 0 0" />
+            <geometry>
+                <mesh filename="package://forklift_robot/forklift_robot_description/meshes/base_link.dae"/>
+            </geometry>
+</xacro:if>
         </collision>
         <xacro:inertial_box m="${base_mass}"  d="${base_length}" w="${base_width}" h="${base_height}"/>
@@ -38,5 +53,5 @@
     <xacro:wheel prefix="left" wheel_radius_multiple="1" />
     <xacro:wheel prefix="right" wheel_radius_multiple="1" />
-    <xacro:wheel prefix="frictionless_back_left" wheel_radius_multiple="1" />
+    <xacro:wheel prefix="frictionless_back_left" wheel_radius_multiple="0.99" />
     <xacro:wheel prefix="frictionless_back_right" wheel_radius_multiple="0.99" />
     <xacro:wheel prefix="frictionless_front_left" wheel_radius_multiple="0.99" />

File: simulation/infobot_agent/urdf/properties.xacro (robot description, xacro)
@@ -1,5 +1,6 @@
 <?xml version="1.0"?>
 <robot xmlns:xacro="http://ros.org/wiki/xacro">
-    <!--GOPAL 400 :  https://www.mobile-robots.de/files/554/factsheet-mr-robotize-gopal-400-e24-09-22-en-min.pdf -->
+<!-- GOPAL400 and FORKLIFT -->
+<xacro:property name="robot_type" value="FORKLIFT"/>
     <xacro:property name="base_length" value="1.4"/>
     <xacro:property name="base_width" value="0.86"/> <!-- wheel_separation -->
@@ -19,3 +20,22 @@
     <xacro:property name="infobot_slip" value="0.0"/>
     <xacro:property name="infobot_damping" value="0.7"/>
+    <xacro:property name="infobot_slide_range" value="2"/>
+<xacro:if value="${robot_type == 'GOPAL400'}">
+    <!--GOPAL 400 :  https://www.mobile-robots.de/files/554/factsheet-mr-robotize-gopal-400-e24-09-22-en-min.pdf -->
+    <xacro:property name="fork_size_x" value="1.2"/>
+    <xacro:property name="fork_size_y" value="0.1"/>
+    <xacro:property name="fork_size_z" value="0.1"/>
+    <xacro:property name="fork_pos_x" value="0.0"/>
+    <xacro:property name="fork_separation" value="0.2"/>
+    <xacro:property name="fork_pos_z" value="0.0"/>
+</xacro:if>
+<xacro:if value="${robot_type == 'FORKLIFT'}">
+    <!-- FORKLIFT -->
+    <xacro:property name="fork_size_x" value="1.2"/>
+    <xacro:property name="fork_size_y" value="0.1"/>
+    <xacro:property name="fork_size_z" value="0.1"/>
+    <xacro:property name="fork_pos_x" value="1.3"/>
+    <xacro:property name="fork_separation" value="0.2"/>
+    <xacro:property name="fork_pos_z" value="-0.3"/>
+</xacro:if>
 </robot>

File: simulation/static_agent_launcher/description/agents.urdf.xacro (robot description, xacro)
@@ -16,7 +16,6 @@
         <child link="base_link"/>
     </joint>
-    <xacro:camera number="1" x="9" y="1" z="7" r="0" p="${pi/4}" yw="${pi/2}"/>
-    <xacro:camera number="2" x="10" y="15" z="6" r="0" p="${pi/4}" yw="${-pi/2}"/>
-    <xacro:aruco number="1" x="9" y="9" z="0.001" r="0" p="0" yw="0"/>
-    <xacro:aruco number="2" x="8" y="6" z="0.001" r="0" p="0" yw="0"/>
+    <xacro:include filename="camera_config.xacro" />
+    <xacro:aruco number="1" x="9" y="9" z="0.001" r="0" p="0" w="0"/>
+    <xacro:aruco number="2" x="8" y="6" z="0.001" r="0" p="0" w="0"/>
 </robot>

File: simulation/static_agent_launcher/description/aruco_macros.xacro (robot description, xacro)
@@ -11,7 +11,7 @@
         <xacro:inertial_box mass="0.1" x="0.12" y="0.15" z="0.15"/>
     </xacro:macro>
-    <xacro:macro name="aruco_joint" params="attach_to number x y z r p yw">
+    <xacro:macro name="aruco_joint" params="attach_to number x y z r p w">
         <joint name="aruco_${number}_joint" type="fixed">
-            <origin xyz="${x} ${y} ${z}" rpy="${r} ${p} ${yw}"/>
+            <origin xyz="${x} ${y} ${z}" rpy="${r} ${p} ${w}"/>
             <parent link="${attach_to}"/>
             <child link="aruco_${number}_link"/>
@@ -46,10 +46,10 @@
         </gazebo>
    </xacro:macro>
-   <xacro:macro name="aruco" params="number x y z r p yw">
-        <xacro:attach_aruco attach_to="base_link" number="${number}" x="${x}" y="${y}" z="${z}" r="${r}" p="${p}" yw="${yw}"/>
+   <xacro:macro name="aruco" params="number x y z r p w">
+        <xacro:attach_aruco attach_to="base_link" number="${number}" x="${x}" y="${y}" z="${z}" r="${r}" p="${p}" w="${w}"/>
    </xacro:macro>
-    <xacro:macro name="attach_aruco" params="attach_to number x y z r p yw">
+    <xacro:macro name="attach_aruco" params="attach_to number x y z r p w">
             <xacro:aruco_link number="${number}"/>
-            <xacro:aruco_joint attach_to="${attach_to}" number="${number}" x="${x}" y="${y}" z="${z}" r="${r}" p="${p}" yw="${yw}"/>
+            <xacro:aruco_joint attach_to="${attach_to}" number="${number}" x="${x}" y="${y}" z="${z}" r="${r}" p="${p}" w="${w}"/>
             <xacro:aruco_gazebo number="${number}"/>
     </xacro:macro>

File: simulation/static_agent_launcher/description/camera_macros.xacro (robot description, xacro)
@@ -17,22 +17,22 @@
         <xacro:inertial_box mass="0.1" x="0.12" y="0.15" z="0.15"/>
     </xacro:macro>
-    <xacro:macro name="camera_joint" params="number x y z r p yw">
+    <xacro:macro name="camera_joint" params="number x y z r p w">
         <joint name="camera_${number}_joint" type="fixed">
-            <origin xyz="${x} ${y} ${z}" rpy="${r} ${p} ${yw}"/>
+            <origin xyz="${x} ${y} ${z}" rpy="${r} ${p} ${w}"/>
             <parent link="base_link"/>
             <child link="camera_${number}_link"/>
         </joint>
     </xacro:macro>
-    <xacro:macro name="camera_gazebo" params="number">
+    <xacro:macro name="camera_gazebo" params="number width height k1 k2 k3 p1 p2 horizental_fov">
         <gazebo reference="camera_${number}_link">
             <sensor name="camera_${number}" type="camera">
                 <always_on>true</always_on>
                 <visualize>true</visualize>
-                <update_rate>30</update_rate>
+                <update_rate>1</update_rate>
                 <camera name="intel_realsense_r200">
-                  <horizontal_fov>1.02974</horizontal_fov>
+                  <horizontal_fov>${horizental_fov}</horizontal_fov>
                   <image>
-                    <width>1920</width>
-                    <height>1080</height>
+                    <width>${width}</width>
+                    <height>${height}</height>
                     <format>R8G8B8</format>
                   </image>
@@ -43,23 +43,24 @@
                   <noise>
                     <type>gaussian</type>
-                    <!-- Noise is sampled independently per pixel on each frame.
-                          That pixel's noise value is added to each of its color
-                          channels, which at that point lie in the range [0,1]. -->
                     <mean>0.0</mean>
                     <stddev>0.007</stddev>
                   </noise>
+                    <distortion>
+                        <k1>${k1}</k1>
+                        <k2>${k2}</k2>
+                        <k3>${k3}</k3>
+                        <p1>${p1}</p1>
+                        <p2>${p2}</p2>
+                    </distortion>
                 </camera>
                   <plugin name="camera_driver_${number}" filename="libgazebo_ros_camera.so">
-                    <!-- camera_name>omit so it defaults to sensor name</camera_name-->
-                    <!-- frame_name>omit so it defaults to link name</frameName-->
-                    <!-- <hack_baseline>0.07</hack_baseline> -->
                   </plugin>
               </sensor>
         </gazebo>
     </xacro:macro>
-    <xacro:macro name="camera" params="number x y z r p yw">
+    <xacro:macro name="camera" params="number x y z r p w width height k1 k2 k3 p1 p2 horizental_fov">
         <xacro:camera_link number="${number}"/>
-        <xacro:camera_joint number="${number}" x="${x}" y="${y}" z="${z}" r="${r}" p="${p}" yw="${yw}"/>
-        <xacro:camera_gazebo number="${number}"/>
+        <xacro:camera_joint number="${number}" x="${x}" y="${y}" z="${z}" r="${r}" p="${p}" w="${w}"/>
+        <xacro:camera_gazebo number="${number}" width="${width}" height="${height}"    k1="${k1}" k2="${k2}" k3="${k3}" p1="${p1}" p2="${p2}" horizental_fov="${horizental_fov}"  />
     </xacro:macro>
 </robot>

Commit message: feat: ci/cd, central command script, scenario runner

File: simulation/infobot_agent/urdf/infobot.gazebo.xacro (robot description, xacro)
@@ -88,5 +88,5 @@
       <sensor name="hls_lfcd_lds" type="ray">
         <always_on>true</always_on>
-        <visualize>true</visualize>
+        <visualize>false</visualize>
         <pose>0 0 0.6 0 0 0</pose>
         <update_rate>5</update_rate>

File: simulation/infobot_agent/urdf/properties.xacro (robot description, xacro)
@@ -2,5 +2,5 @@
 <robot xmlns:xacro="http://ros.org/wiki/xacro">
 <!-- GOPAL400 and FORKLIFT -->
-<xacro:property name="robot_type" value="GOPAL400"/>
+<xacro:property name="robot_type" value="FORKLIFT"/>
     <xacro:property name="base_length" value="1.4"/>
     <xacro:property name="base_width" value="0.86"/> <!-- wheel_separation -->

File: simulation/static_agent_launcher/description/camera_config.xacro (robot description, xacro)
@@ -2,8 +2,10 @@
 <!-- =================================== -->
 <robot xmlns:xacro="http://www.ros.org/wiki/xacro">
+<!--
 <xacro:camera number="160" x="-23.768993347281643" y="1.0959115856381252" z="7.792710237230576" r="-3.072200475262292" p="2.0401256682927498" w="3.1384164986805017" width="2160" height="3840" k1="-0.3990864717265948" k2="0.2016451846353012" k3="-0.053753317426588856" p1="-0.00013457492654973615" p2="0.0003788431220127677" horizental_fov="0.9062245961423843" aspect_ratio="0.6346135746416991"  />
 <xacro:camera number="161" x="-15.54857444861928" y="1.1875803973838794" z="8.430721825553768" r="3.1401165362282915" p="1.8467776536834755" w="-3.075174579490206" width="2160" height="3840" k1="-0.5337684959685228" k2="0.34369206124627594" k3="-0.11312322233867529" p1="-0.001568761626559521" p2="0.0012933658245218613" horizental_fov="0.7979068207653639" aspect_ratio="0.6219373044342069"  />
 <xacro:camera number="162" x="-5.583158189893618" y="1.1215696998181661" z="7.334558192411434" r="-3.121470473216963" p="1.882414969291388" w="3.1315374728737932" width="2160" height="3840" k1="-0.3881529379410545" k2="0.21282043348416652" k3="-0.07191487688493671" p1="7.348232914337802e-05" p2="-0.0003723515252576787" horizental_fov="0.934637563021535" aspect_ratio="0.6380980311690627"  />
 <xacro:camera number="163" x="6.408863223463874" y="1.0584660310604614" z="7.292500745934433" r="-3.1247537437337134" p="1.6132230097420674" w="3.072926607602098" width="2160" height="3840" k1="-0.38583566587127305" k2="0.2099961443873393" k3="-0.07094931776988343" p1="0.00014849011979552266" p2="9.279371221442497e-05" horizental_fov="0.9312481766450852" aspect_ratio="0.6378137006195269"  />
+-->
 <xacro:camera number="164" x="19.018611699231805" y="0.5996158690202326" z="7.312413251033551" r="3.0865049949744816" p="1.2064798251635096" w="-0.10259603486110593" width="2160" height="3840" k1="-0.3851544658419547" k2="0.2065606446662026" k3="-0.06703301309031716" p1="-0.0002282099854856601" p2="-8.882469357164693e-05" horizental_fov="0.9343447506168914" aspect_ratio="0.6383050770452745"  />
 <xacro:camera number="165" x="19.780977546074062" y="-3.598892158741938" z="7.320450325717852" r="3.092351302733551" p="1.9069402784416059" w="-1.63895299731986" width="2160" height="3840" k1="-0.3856199901471728" k2="0.20812766168662827" k3="-0.0686518264523881" p1="-8.229104930400743e-05" p2="-0.00023961544692403472" horizental_fov="0.9339854982138229" aspect_ratio="0.6382418389072573"  />
@@ -11,6 +13,8 @@
 <xacro:camera number="167" x="20.320795688398483" y="8.551222492793519" z="7.698006516690173" r="-2.864067809004126" p="1.6165247062294361" w="3.049326481704911" width="2160" height="3840" k1="-0.3838819131967851" k2="0.2010505063378464" k3="-0.062406328638322184" p1="-0.0001711681317662323" p2="-0.0001384477473404489" horizental_fov="0.9326674829664602" aspect_ratio="0.6380360618380091"  />
 <xacro:camera number="168" x="26.79180252096381" y="5.716299217374743" z="3.8958341874803013" r="2.0879686599511014" p="1.5484721682976101" w="0.02430880840685812" width="2160" height="3840" k1="-0.38226542199738556" k2="0.19688945293158802" k3="-0.05884113267485558" p1="-0.00019454336997989425" p2="0.00010222372875181348" horizental_fov="0.930340781288024" aspect_ratio="0.6377205101360616"  />
+<!--
 <xacro:camera number="169" x="30.084965589192375" y="9.359551955197704" z="5.17974502700982" r="-2.6817009758316908" p="1.442123361726637" w="-3.087108573615953" width="2160" height="3840" k1="-0.376908078697939" k2="0.1841695668036844" k3="-0.05236396951447785" p1="-0.0006789329541068425" p2="-0.0003816943552840085" horizental_fov="0.9306534293111707" aspect_ratio="0.6373718963712801"  />
 <xacro:camera number="170" x="36.82995339051741" y="9.404901482485904" z="5.154350415603337" r="-2.66777470309351" p="1.5376363780888378" w="-3.089363397883026" width="2160" height="3840" k1="-0.3840696848810335" k2="0.20309686574554098" k3="-0.06443293775304995" p1="-0.0002648898125099341" p2="0.00011495455326132926" horizental_fov="0.9336309514986754" aspect_ratio="0.6382016868830621"  />
 <xacro:camera number="171" x="42.4426904656032" y="9.38157274756824" z="5.146596979178394" r="-2.7448623326295176" p="1.5704089535445784" w="-3.132973283776775" width="2160" height="3840" k1="-0.3840696848810335" k2="0.20309686574554098" k3="-0.06443293775304995" p1="-0.0002648898125099341" p2="0.00011495455326132926" horizental_fov="0.9336309514986754" aspect_ratio="0.6382016868830621"  />
+-->
 </robot>
