Commit message: improve simulation (infobot), improve dev environment (docker), cleanup the startup scripts, fix issue with camera configs

File: simulation/infobot_agent/urdf/links.xacro (robot description, xacro)
@@ -7,5 +7,5 @@
             <origin xyz="0 0 0" rpy="0 0 0" />
             <geometry>
-                <mesh filename="file://infobot_agent/models/infobot_common/meshes/AMR_GP400.dae" scale="1 1 1"/>
+                <mesh filename="package://infobot_common/meshes/AMR_GP400.dae" scale="1 1 1"/>
                 <!-- <box size="${base_length} ${base_width} ${base_height}" /> -->
             </geometry>
@@ -21,5 +21,5 @@
 <xacro:if value="${robot_type == 'GOPAL400'}">
             <geometry>
-                <mesh filename="file://infobot_agent/models/infobot_common/meshes/AMR_GP400.dae" scale="1 1 1"/>
+                <mesh filename="package://infobot_common/meshes/AMR_GP400.dae" scale="1 1 1"/>
                 <!-- <box size="${base_length} ${base_width} ${base_height}" />  -->
             </geometry>

File: simulation/infobot_agent/urdf/sensors.xacro (robot description, xacro)
@@ -16,5 +16,5 @@
       <origin xyz="0 0 0" rpy="0 0 0"/>
       <geometry>
-        <mesh filename="file://infobot_agent/models/infobot_common/meshes/lds.dae" scale="0.001 0.001 0.001"/>
+        <mesh filename="package://infobot_common/meshes/lds.dae" scale="0.001 0.001 0.001"/>
       </geometry>
       <material name="dark"/>
@@ -30,5 +30,5 @@
      <origin xyz="0 0 0" rpy="0 0 ${pi/2}"/>
       <geometry>
-       <mesh filename="file://infobot_agent/models/infobot_common/meshes/camera.dae" scale="1 1 1" />
+       <mesh filename="package://infobot_common/meshes/camera.dae" scale="1 1 1" />
       </geometry>
     </visual>

Commit message: fix: infobot mesh link error

File: simulation/infobot_agent/urdf/links.xacro (robot description, xacro)
@@ -7,5 +7,5 @@
             <origin xyz="0 0 0" rpy="0 0 0" />
             <geometry>
-                <mesh filename="package://infobot_common/meshes/AMR_GP400.dae" scale="1 1 1"/>
+                <mesh filename="file://$(find infobot_agent)/models/infobot_common/meshes/AMR_GP400.dae" scale="1 1 1"/>
                 <!-- <box size="${base_length} ${base_width} ${base_height}" /> -->
             </geometry>
@@ -14,5 +14,5 @@
             <origin xyz="-1.5 -0.5 0" rpy="0 0 0" />
             <geometry>
-                <mesh filename="package://forklift_robot/forklift_robot_description/meshes/base_link.dae"/>
+                <mesh filename="file://$(find simlan_gazebo_environment)/models/forklift_robot/forklift_robot_description/meshes/base_link.dae"/>
             </geometry>
 </xacro:if>
@@ -21,5 +21,5 @@
 <xacro:if value="${robot_type == 'GOPAL400'}">
             <geometry>
-                <mesh filename="package://infobot_common/meshes/AMR_GP400.dae" scale="1 1 1"/>
+                <mesh filename="file://$(find infobot_agent)/models/infobot_common/meshes/AMR_GP400.dae" scale="1 1 1"/>
                 <!-- <box size="${base_length} ${base_width} ${base_height}" />  -->
             </geometry>
@@ -28,5 +28,5 @@
             <origin xyz="-1.5 -0.5 0" rpy="0 0 0" />
             <geometry>
-                <mesh filename="package://forklift_robot/forklift_robot_description/meshes/base_link.dae"/>
+                <mesh filename="file://$(find simlan_gazebo_environment)/models/forklift_robot/forklift_robot_description/meshes/base_link.dae"/>
             </geometry>
 </xacro:if>

File: simulation/infobot_agent/urdf/sensors.xacro (robot description, xacro)
@@ -16,5 +16,5 @@
       <origin xyz="0 0 0" rpy="0 0 0"/>
       <geometry>
-        <mesh filename="package://infobot_common/meshes/lds.dae" scale="0.001 0.001 0.001"/>
+        <mesh filename="file://$(find infobot_agent)/models/infobot_common/meshes/lds.dae" scale="0.001 0.001 0.001"/>
       </geometry>
       <material name="dark"/>
@@ -30,5 +30,5 @@
      <origin xyz="0 0 0" rpy="0 0 ${pi/2}"/>
       <geometry>
-       <mesh filename="package://infobot_common/meshes/camera.dae" scale="1 1 1" />
+       <mesh filename="file://$(find infobot_agent)/models/infobot_common/meshes/camera.dae" scale="1 1 1" />
       </geometry>
     </visual>

Commit message: feat: delivery 1.0.5

File: simulation/infobot_agent/urdf/links.xacro (robot description, xacro)
@@ -7,5 +7,5 @@
             <origin xyz="0 0 0" rpy="0 0 0" />
             <geometry>
-                <mesh filename="file://$(find infobot_agent)/models/infobot_common/meshes/AMR_GP400.dae" scale="1 1 1"/>
+                <mesh filename="package://infobot_common/meshes/AMR_GP400.dae" scale="1 1 1"/>
                 <!-- <box size="${base_length} ${base_width} ${base_height}" /> -->
             </geometry>
@@ -14,5 +14,5 @@
             <origin xyz="-1.5 -0.5 0" rpy="0 0 0" />
             <geometry>
-                <mesh filename="file://$(find simlan_gazebo_environment)/models/forklift_robot/forklift_robot_description/meshes/base_link.dae"/>
+                <mesh filename="package://forklift_robot/forklift_robot_description/meshes/base_link.dae"/>
             </geometry>
 </xacro:if>
@@ -21,5 +21,5 @@
 <xacro:if value="${robot_type == 'GOPAL400'}">
             <geometry>
-                <mesh filename="file://$(find infobot_agent)/models/infobot_common/meshes/AMR_GP400.dae" scale="1 1 1"/>
+                <mesh filename="package://infobot_common/meshes/AMR_GP400.dae" scale="1 1 1"/>
                 <!-- <box size="${base_length} ${base_width} ${base_height}" />  -->
             </geometry>
@@ -28,5 +28,5 @@
             <origin xyz="-1.5 -0.5 0" rpy="0 0 0" />
             <geometry>
-                <mesh filename="file://$(find simlan_gazebo_environment)/models/forklift_robot/forklift_robot_description/meshes/base_link.dae"/>
+                <mesh filename="package://forklift_robot/forklift_robot_description/meshes/base_link.dae"/>
             </geometry>
 </xacro:if>

File: simulation/infobot_agent/urdf/sensors.xacro (robot description, xacro)
@@ -16,5 +16,5 @@
       <origin xyz="0 0 0" rpy="0 0 0"/>
       <geometry>
-        <mesh filename="file://$(find infobot_agent)/models/infobot_common/meshes/lds.dae" scale="0.001 0.001 0.001"/>
+        <mesh filename="package://infobot_common/meshes/lds.dae" scale="0.001 0.001 0.001"/>
       </geometry>
       <material name="dark"/>
@@ -30,5 +30,5 @@
      <origin xyz="0 0 0" rpy="0 0 ${pi/2}"/>
       <geometry>
-       <mesh filename="file://$(find infobot_agent)/models/infobot_common/meshes/camera.dae" scale="1 1 1" />
+       <mesh filename="package://infobot_common/meshes/camera.dae" scale="1 1 1" />
       </geometry>
     </visual>
